File: right/right.sch (KiCad schematic (older format))
At the start: 52 parts, among them J1 Modulo-Jack, J2 Modulo-Jack, J3 Modulo-Jack, SW1 SW_Push, SW10 SW_Push, SW11 SW_Push, SW12 SW_Push, SW13 SW_Push, SW14 SW_Push, SW15 SW_Push, SW16 SW_Push, SW17 SW_Push, SW18 SW_Push, SW19 SW_Push, SW2 SW_Push, SW20 SW_Push, SW21 SW_Push, SW22 SW_Push, SW23 SW_Push, SW24 SW_Push, SW25 SW_Push, SW26 SW_Push, SW27 SW_Push, SW28 SW_Push, SW29 SW_Push, SW3 SW_Push, SW30 SW_Push, SW31 SW_Push, SW32 SW_Push, SW33 SW_Push, SW34 SW_Push, SW35 SW_Push, SW36 SW_Push, SW37 SW_Push, SW38 SW_Push, SW39 SW_Push, SW4 SW_Push, SW40 SW_Push, SW41 SW_Push, SW42 SW_Push, SW43 SW_Push, SW5 SW_Push, SW6 SW_Push, SW7 SW_Push, SW8 SW_Push, SW9 SW_Push, U1 MCP23017_SP, U2 MCP23017_SP, U3 MCP23017_SP

Commit message: last commit
Parts:
- added SW44: SW_DPDT_x2, lib:SlideSwitch_IS2235, symbol Switch:SW_DPDT_x2
Connections:
- net GND: now also SW44.3 (C)
- net VCC: now also SW44.1 (A); no longer U1.17 (A2), U2.17 (A2), U3.17 (A2)
- new net ADDR: SW44.2 (B), U1.17 (A2), U2.17 (A2), U3.17 (A2)
- no-connect marks 19 -> 22
Changed lines of the file:
@@
 Wire Wire Line
 	1000 5450 1000 5000
-Text GLabel 4850 5950 3    50   Output ~ 0
-ADDR
-$Comp
-L power:VCC #PWR057
-U 1 1 5D145BAD
-P 4850 5950
-F 0 "#PWR057" H 4850 5800 50  0001 C CNN
-F 1 "VCC" H 4867 6123 50  0000 C CNN
-F 2 "" H 4850 5950 50  0001 C CNN
-F 3 "" H 4850 5950 50  0001 C CNN
-	1    4850 5950
-	1    0    0    -1
-$EndComp
 $Comp
 L Device:C C1
@@
 	1    0    0    -1
 $EndComp
+$Comp
+L Switch:SW_DPDT_x2 SW44
+U 1 1 5CF9A790
+P 2250 6800
+F 0 "SW44" H 2250 7085 50  0000 C CNN
+F 1 "SW_DPDT_x2" H 2250 6994 50  0000 C CNN
+F 2 "lib:SlideSwitch_IS2235" H 2250 6800 50  0001 C CNN
+F 3 "~" H 2250 6800 50  0001 C CNN
+	1    2250 6800
+	1    0    0    -1
+$EndComp
+$Comp
+L Switch:SW_DPDT_x2 SW44
+U 2 1 5CF9B03C
+P 2250 7350
+F 0 "SW44" H 2250 7635 50  0000 C CNN
+F 1 "SW_DPDT_x2" H 2250 7544 50  0000 C CNN
+F 2 "lib:SlideSwitch_IS2235" H 2250 7350 50  0001 C CNN
+F 3 "~" H 2250 7350 50  0001 C CNN
+	2    2250 7350
+	1    0    0    -1
+$EndComp
+NoConn ~ 2050 7350
+NoConn ~ 2450 7250
+NoConn ~ 2450 7450
+Text GLabel 2050 6800 0    50   Output ~ 0
+ADDR
+$Comp
+L power:VCC #PWR058
+U 1 1 5CFA3438
+P 2450 6700
+F 0 "#PWR058" H 2450 6550 50  0001 C CNN
+F 1 "VCC" H 2467 6873 50  0000 C CNN
+F 2 "" H 2450 6700 50  0001 C CNN
+F 3 "" H 2450 6700 50  0001 C CNN
+	1    2450 6700
+	1    0    0    -1
+$EndComp
+$Comp
+L power:GND #PWR062
+U 1 1 5CFA38DB
+P 2450 6900
+F 0 "#PWR062" H 2450 6650 50  0001 C CNN
+F 1 "GND" H 2455 6727 50  0000 C CNN
+F 2 "" H 2450 6900 50  0001 C CNN
+F 3 "" H 2450 6900 50  0001 C CNN
+	1    2450 6900
+	1    0    0    -1
+$EndComp
+$Comp
+L power:VCC #PWR057
+U 1 1 5CFB8183
+P 4650 5950
+F 0 "#PWR057" H 4650 5800 50  0001 C CNN
+F 1 "VCC" H 4667 6123 50  0000 C CNN
+F 2 "" H 4650 5950 50  0001 C CNN
+F 3 "" H 4650 5950 50  0001 C CNN
+	1    4650 5950
+	1    0    0    -1
+$EndComp
+$Comp
+L power:GND #PWR063
+U 1 1 5CFB88EB
+P 5200 6000
+F 0 "#PWR063" H 5200 5750 50  0001 C CNN
+F 1 "GND" H 5205 5827 50  0000 C CNN
+F 2 "" H 5200 6000 50  0001 C CNN
+F 3 "" H 5200 6000 50  0001 C CNN
+	1    5200 6000
+	1    0    0    -1
+$EndComp
+$Comp
+L power:PWR_FLAG #FLG01
+U 1 1 5CFB8FF5
+P 4650 5950
+F 0 "#FLG01" H 4650 6025 50  0001 C CNN
+F 1 "PWR_FLAG" H 4650 6123 50  0000 C CNN
+F 2 "" H 4650 5950 50  0001 C CNN
+F 3 "~" H 4650 5950 50  0001 C CNN
+	1    4650 5950
+	1    0    0    1
+$EndComp
+$Comp
+L power:PWR_FLAG #FLG02
+U 1 1 5CFB94E7
+P 5200 6000
+F 0 "#FLG02" H 5200 6075 50  0001 C CNN
+F 1 "PWR_FLAG" H 5200 6173 50  0000 C CNN
+F 2 "" H 5200 6000 50  0001 C CNN
+F 3 "~" H 5200 6000 50  0001 C CNN
+	1    5200 6000
+	1    0    0    -1
+$EndComp
+$Comp
+L power:PWR_FLAG #FLG03
+U 1 1 5CFBC593
+P 5650 6000
+F 0 "#FLG03" H 5650 6075 50  0001 C CNN
+F 1 "PWR_FLAG" H 5650 6173 50  0000 C CNN
+F 2 "" H 5650 6000 50  0001 C CNN
+F 3 "~" H 5650 6000 50  0001 C CNN
+	1    5650 6000
+	1    0    0    -1
+$EndComp
+Text GLabel 5650 6000 3    50   Input ~ 0
+SCK
 $EndSCHEMATC

Commit message: modify right to JIS layout
Parts:
- removed SW32: SW_Push, MX_Socket:MXOnly-1U-Hotswap, symbol Switch:SW_Push
- removed SW39: SW_Push, MX_Socket:MXOnly-2U-Hotswap, symbol Switch:SW_Push
- removed SW40: SW_Push, MX_Socket:MXOnly-1.5U-Hotswap, symbol Switch:SW_Push
- removed SW41: SW_Push, MX_Socket:MXOnly-2.25U-Hotswap, symbol Switch:SW_Push
- removed SW42: SW_Push, MX_Socket:MXOnly-2.75U-Hotswap, symbol Switch:SW_Push
- removed SW43: SW_Push, MX_Socket:MXOnly-2U-Hotswap-ReversedStabilizers, symbol Switch:SW_Push
- SW34: footprint MX_Socket:MXOnly-1U-Hotswap -> MX_Socket:MXOnly-1.25U-Hotswap
- SW37: footprint MX_Socket:MXOnly-1.25U-Hotswap -> MX_Socket:MXOnly-1U-Hotswap
Connections:
- net GND: now also SW16.1, SW24.1, SW30.1, SW31.1; no longer SW16.2, SW24.2, SW30.2, SW31.2
- net SW1: now also U1.24 (GPA3); no longer U1.2 (GPB1)
- net SW10: now also U1.8 (GPB7); no longer U1.7 (GPB6)
- net SW11: now also U1.21 (GPA0); no longer U1.5 (GPB4)
- net SW12: now also U1.7 (GPB6); no longer U1.22 (GPA1)
- net SW13: now also U1.22 (GPA1); no longer U1.4 (GPB3)
- net SW14: now also U1.6 (GPB5); no longer U1.23 (GPA2)
- net SW15: now also U1.23 (GPA2); no longer U2.28 (GPA7)
- net SW16: now also SW16.2, U1.5 (GPB4); no longer SW16.1, U1.6 (GPB5)
- net SW17: now also U2.28 (GPA7); no longer U2.1 (GPB0)
- net SW18: now also U3.28 (GPA7); no longer U3.26 (GPA5)
- net SW19: now also U2.25 (GPA4); no longer U3.2 (GPB1)
- net SW2: now also U1.4 (GPB3); no longer U1.25 (GPA4)
- net SW20: now also U2.3 (GPB2); no longer U3.27 (GPA6)
- net SW21: now also U2.26 (GPA5); no longer U2.2 (GPB1)
- net SW22: now also U2.2 (GPB1); no longer U2.27 (GPA6)
- net SW23: now also U2.27 (GPA6); no longer U1.8 (GPB7)
- net SW24: now also SW24.2, U2.1 (GPB0); no longer SW24.1, U2.26 (GPA5)
- net SW26: now also U3.25 (GPA4); no longer U3.4 (GPB3)
- net SW27: now also U3.3 (GPB2); no longer U3.1 (GPB0)
- net SW28: now also U3.26 (GPA5); no longer U3.28 (GPA7)
- net SW29: now also U3.2 (GPB1); no longer U2.3 (GPB2)
- net SW3: now also U1.25 (GPA4); no longer U1.26 (GPA5)
- net SW30: now also SW30.2, U3.1 (GPB0); no longer SW30.1, U3.25 (GPA4)
- net SW31: now also SW31.2, U3.27 (GPA6); no longer SW31.1, U3.3 (GPB2)
- net SW4: now also U1.3 (GPB2); no longer U1.27 (GPA6)
- net SW5: now also U1.26 (GPA5); no longer U1.28 (GPA7)
- net SW6: now also U1.2 (GPB1); no longer U1.21 (GPA0)
- net SW7: now also U1.27 (GPA6); no longer U1.3 (GPB2)
- net SW8: now also U1.1 (GPB0); no longer U1.24 (GPA3)
- net SW9: now also U1.28 (GPA7); no longer U1.1 (GPB0)
- net SW32: no longer names the net of U3.8 (GPB7)
- no-connect marks 22 -> 23
Changed lines of the file:
@@
 F 3 "~" H 5500 2200 50  0001 C CNN
 	1    5500 2000
-	1    0    0    -1
+	-1   0    0    -1
 $EndComp
 $Comp
@@
 F 3 "~" H 5500 3200 50  0001 C CNN
 	1    5500 3000
-	1    0    0    -1
+	-1   0    0    -1
 $EndComp
 $Comp
@@
 F 3 "~" H 4800 4200 50  0001 C CNN
 	1    4800 4000
-	1    0    0    -1
+	-1   0    0    -1
 $EndComp
 $Comp
@@
 F 3 "~" H 5500 4200 50  0001 C CNN
 	1    5500 4000
-	1    0    0    -1
+	-1   0    0    -1
 $EndComp
 $Comp
@@
 $EndComp
 $Comp
-L Switch:SW_Push SW32
-U 1 1 5CF5C6F4
-P 1200 5000
-F 0 "SW32" H 1200 5285 50  0000 C CNN
-F 1 "SW_Push" H 1200 5194 50  0000 C CNN
-F 2 "MX_Socket:MXOnly-1U-Hotswap" H 1200 5200 50  0001 C CNN
-F 3 "~" H 1200 5200 50  0001 C CNN
-	1    1200 5000
-	1    0    0    -1
-$EndComp
-$Comp
-L power:GND #PWR032
-U 1 1 5CF5C6FA
-P 1400 5450
-F 0 "#PWR032" H 1400 5200 50  0001 C CNN
-F 1 "GND" H 1405 5277 50  0000 C CNN
-F 2 "" H 1400 5450 50  0001 C CNN
-F 3 "" H 1400 5450 50  0001 C CNN
-	1    1400 5450
-	1    0    0    -1
-$EndComp
-$Comp
 L Switch:SW_Push SW33
 U 1 1 5CF5C700
@@
 F 0 "SW34" H 2650 5285 50  0000 C CNN
 F 1 "SW_Push" H 2650 5194 50  0000 C CNN
-F 2 "MX_Socket:MXOnly-1U-Hotswap" H 2650 5200 50  0001 C CNN
+F 2 "MX_Socket:MXOnly-1.25U-Hotswap" H 2650 5200 50  0001 C CNN
 F 3 "~" H 2650 5200 50  0001 C CNN
 	1    2650 5000
@@
 F 0 "SW37" H 4800 5285 50  0000 C CNN
 F 1 "SW_Push" H 4800 5194 50  0000 C CNN
-F 2 "MX_Socket:MXOnly-1.25U-Hotswap" H 4800 5200 50  0001 C CNN
+F 2 "MX_Socket:MXOnly-1U-Hotswap" H 4800 5200 50  0001 C CNN
 F 3 "~" H 4800 5200 50  0001 C CNN
 	1    4800 5000
@@
 Text GLabel 5300 4000 0    50   Output ~ 0
 SW31
-Text GLabel 1000 5000 0    50   Output ~ 0
-SW32
 Text GLabel 1750 5000 0    50   Output ~ 0
 SW33
@@
 Text GLabel 5300 5000 0    50   Output ~ 0
 SW38
+Text GLabel 9700 1550 2    50   Input ~ 0
+SW1
+Text GLabel 8300 1450 0    50   Input ~ 0
+SW2
+Text GLabel 9700 1450 2    50   Input ~ 0
+SW3
+Text GLabel 8300 1350 0    50   Input ~ 0
+SW4
+Text GLabel 9700 1350 2    50   Input ~ 0
+SW5
 Text GLabel 8300 1250 0    50   Input ~ 0
-SW1
-Text GLabel 9700 1450 2    50   Input ~ 0
-SW2
-Text GLabel 9700 1350 2    50   Input ~ 0
-SW3
+SW6
 Text GLabel 9700 1250 2    50   Input ~ 0
-SW4
-Text GLabel 9700 1150 2    50   Input ~ 0
-SW5
+SW7
+Text GLabel 8300 1150 0    50   Input ~ 0
+SW8
+Text GLabel 8300 1850 0    50   Input ~ 0
+SW10
 Text GLabel 9700 1850 2    50   Input ~ 0
-SW6
-Text GLabel 8300 1350 0    50   Input ~ 0
-SW7
-Text GLabel 9700 1550 2    50   Input ~ 0
-SW8
+SW11
 Text GLabel 8300 1750 0    50   Input ~ 0
-SW10
+SW12
+Text GLabel 9700 1750 2    50   Input ~ 0
+SW13
+Text GLabel 8300 1650 0    50   Input ~ 0
+SW14
+Text GLabel 9700 1650 2    50   Input ~ 0
+SW15
 Text GLabel 8300 1550 0    50   Input ~ 0
-SW11
-Text GLabel 9700 1750 2    50   Input ~ 0
-SW12
-Text GLabel 8300 1450 0    50   Input ~ 0
-SW13
-Text GLabel 9700 1650 2    50   Input ~ 0
-SW14
-Text GLabel 12400 2800 2    50   Input ~ 0
-SW15
-Text GLabel 8300 1650 0    50   Input ~ 0
 SW16
 Text GLabel 8300 2400 0    50   Input ~ 0
@@
 NoConn ~ 9750 5350
 NoConn ~ 9750 5550
+Text GLabel 12400 2800 2    50   Input ~ 0
+SW17
+Text GLabel 9750 4300 2    50   Input ~ 0
+SW18
+Text GLabel 12400 3100 2    50   Input ~ 0
+SW19
+Text GLabel 11000 3000 0    50   Input ~ 0
+SW20
+Text GLabel 12400 3000 2    50   Input ~ 0
+SW21
+Text GLabel 11000 2900 0    50   Input ~ 0
+SW22
+Text GLabel 12400 2900 2    50   Input ~ 0
+SW23
 Text GLabel 11000 2800 0    50   Input ~ 0
-SW17
-Text GLabel 9750 4500 2    50   Input ~ 0
-SW18
-Text GLabel 8350 4400 0    50   Input ~ 0
-SW19
-Text GLabel 9750 4400 2    50   Input ~ 0
-SW20
-Text GLabel 11000 2900 0    50   Input ~ 0
-SW21
-Text GLabel 12400 2900 2    50   Input ~ 0
-SW22
-Text GLabel 8300 1850 0    50   Input ~ 0
-SW23
-Text GLabel 12400 3000 2    50   Input ~ 0
 SW24
 Text GLabel 9750 4700 2    50   Input ~ 0
 SW25
-Text GLabel 8350 4600 0    50   Input ~ 0
-SW26
+Text GLabel 8350 4500 0    50   Input ~ 0
+SW27
+Text GLabel 9750 4500 2    50   Input ~ 0
+SW28
+Text GLabel 10150 3050 0    50   Input ~ 0
+SW29
 Text GLabel 8350 4300 0    50   Input ~ 0
-SW27
-Text GLabel 9750 4300 2    50   Input ~ 0
-SW28
-Text GLabel 11000 3000 0    50   Input ~ 0
-SW29
-Text GLabel 9750 4600 2    50   Input ~ 0
 SW30
-Text GLabel 8350 4500 0    50   Input ~ 0
-SW31
-Text GLabel 8350 5000 0    50   Input ~ 0
-SW32
 Text GLabel 9750 5000 2    50   Input ~ 0
 SW33
-Text GLabel 8350 4900 0    50   Input ~ 0
-SW34
 Text GLabel 9750 4900 2    50   Input ~ 0
 SW35
-Text GLabel 8350 4800 0    50   Input ~ 0
-SW36
 Text GLabel 9750 4800 2    50   Input ~ 0
 SW37
-Text GLabel 8350 4700 0    50   Input ~ 0
-SW38
 Text GLabel 9700 2550 2    50   Input ~ 0
 ADDR
@@
 Wire Wire Line
 	4000 6250 3450 6250
-$Comp
-L Switch:SW_Push SW39
-U 1 1 5D0FD0CA
-P 6950 1400
-F 0 "SW39" H 6950 1685 50  0000 C CNN
-F 1 "SW_Push" H 6950 1594 50  0000 C CNN
-F 2 "MX_Socket:MXOnly-2U-Hotswap" H 6950 1600 50  0001 C CNN
-F 3 "~" H 6950 1600 50  0001 C CNN
-	1    6950 1400
-	1    0    0    -1
-$EndComp
-$Comp
-L Switch:SW_Push SW40
-U 1 1 5D0FD9ED
-P 6250 2400
-F 0 "SW40" H 6250 2685 50  0000 C CNN
-F 1 "SW_Push" H 6250 2594 50  0000 C CNN
-F 2 "MX_Socket:MXOnly-1.5U-Hotswap" H 6250 2600 50  0001 C CNN
-F 3 "~" H 6250 2600 50  0001 C CNN
-	1    6250 2400
-	-1   0    0    -1
-$EndComp
-$Comp
-L Switch:SW_Push SW41
-U 1 1 5D10007D
-P 5500 3400
-F 0 "SW41" H 5500 3685 50  0000 C CNN
-F 1 "SW_Push" H 5500 3594 50  0000 C CNN
-F 2 "MX_Socket:MXOnly-2.25U-Hotswap" H 5500 3600 50  0001 C CNN
-F 3 "~" H 5500 3600 50  0001 C CNN
-	1    5500 3400
-	1    0    0    -1
-$EndComp
-$Comp
-L Switch:SW_Push SW42
-U 1 1 5D100920
-P 5500 4400
-F 0 "SW42" H 5500 4685 50  0000 C CNN
-F 1 "SW_Push" H 5500 4594 50  0000 C CNN
-F 2 "MX_Socket:MXOnly-2.75U-Hotswap" H 5500 4600 50  0001 C CNN
-F 3 "~" H 5500 4600 50  0001 C CNN
-	1    5500 4400
-	-1   0    0    -1
-$EndComp
-$Comp
-L Switch:SW_Push SW43
-U 1 1 5D101884
-P 1200 5450
-F 0 "SW43" H 1200 5735 50  0000 C CNN
-F 1 "SW_Push" H 1200 5644 50  0000 C CNN
-F 2 "MX_Socket:MXOnly-2U-Hotswap-ReversedStabilizers" H 1200 5650 50  0001 C CNN
-F 3 "~" H 1200 5650 50  0001 C CNN
-	1    1200 5450
-	1    0    0    -1
-$EndComp
-Wire Wire Line
-	6750 1000 6750 1400
 Wire Wire Line
 	7150 1400 7150 1000
-Connection ~ 7150 1400
 Wire Wire Line
 	6450 2000 6450 2400
-Connection ~ 6450 2400
-Wire Wire Line
-	6050 2400 6050 2000
-Wire Wire Line
-	5300 3000 5300 3400
 Wire Wire Line
 	5700 3400 5700 3000
-Connection ~ 5700 3400
-Wire Wire Line
-	5300 4000 5300 4400
 Wire Wire Line
 	5700 4400 5700 4000
-Connection ~ 5700 4400
-Wire Wire Line
-	1400 5000 1400 5450
-Connection ~ 1400 5450
-Wire Wire Line
-	1000 5450 1000 5000
 $Comp
 L Device:C C1
@@
 	1    0    0    -1
 $EndComp
-Text GLabel 8300 1150 0    50   Input ~ 0
+Text GLabel 9700 1150 2    50   Input ~ 0
 SW9
 $Comp
@@
 NoConn ~ 11000 3400
 NoConn ~ 11000 3500
-NoConn ~ 12400 3100
 NoConn ~ 12400 3200
 NoConn ~ 12400 3300
@@
 Text GLabel 5650 6000 3    50   Input ~ 0
 SCK
+NoConn ~ 8350 5000
+Text GLabel 8350 4700 0    50   Input ~ 0
+SW38
+Text GLabel 8350 4800 0    50   Input ~ 0
+SW36
+Text GLabel 8350 4900 0    50   Input ~ 0
+SW34
+Text GLabel 9750 4400 2    50   Input ~ 0
+SW31
+Text GLabel 9750 4600 2    50   Input ~ 0
+SW26
+Text GLabel 8350 4400 0    50   Input ~ 0
+SW29
+NoConn ~ 8350 4600
 $EndSCHEMATC
