File: left/left.kicad_pcb (KiCad board)
At the start: 2 copper layers, 168.6 x 104.5 mm, 53 parts, among them J1 Modulo-Jack, J2 Modulo-Jack, J3 Modulo-Jack, SW1 SW_Push, SW10 SW_Push, SW11 SW_Push, SW12 SW_Push, SW13 SW_Push, SW14 SW_Push, SW15 SW_Push, SW16 SW_Push, SW17 SW_Push, SW18 SW_Push, SW19 SW_Push, SW2 SW_Push, SW20 SW_Push, SW21 SW_Push, SW22 SW_Push, SW23 SW_Push, SW24 SW_Push, SW25 SW_Push, SW26 SW_Push, SW27 SW_Push, SW28 SW_Push, SW29 SW_Push, SW3 SW_Push, SW30 SW_Push, SW31 SW_Push, SW32 SW_Push, SW4 SW_Push, SW5 SW_Push, SW50 SW_DPDT_x2, SW51 SW_DPDT_x2, SW6 SW_Push, SW7 SW_Push, SW8 SW_Push, SW9 SW_Push, U1 MCP23017_SP, U2 MCP23017_SP

Commit message: move screw
Parts:
- moved ? 19.0 mm to (185.2, 133.0)
Routing:
- net GND: track 1070.6 -> 1072.6 mm
Changed lines of the file:
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@@
   )
   (module lib:MountingHole_2.2mm_M2 locked (layer F.Cu)
-    (at 166.25 133)
+    (at 185.25 133)
     (descr "Mounting Hole 2.2mm, no annular, M2")
     (tags "mounting hole 2.2mm no annular m2")
@@
   (segment (start 210.092 130.268) (end 210.092 132.622) (width 0.5) (layer B.Cu) (net 1))
   (segment (start 210.092 132.622) (end 215.265 137.795) (width 0.5) (layer B.Cu) (net 1))
-  (segment (start 182.88 134.62) (end 185.42 134.62) (width 0.5) (layer B.Cu) (net 1))
-  (segment (start 182.88 134.62) (end 183.515 134.62) (width 0.5) (layer B.Cu) (net 1))
-  (segment (start 189.772 130.268) (end 210.092 130.268) (width 0.5) (layer B.Cu) (net 1))
-  (segment (start 185.42 134.62) (end 189.772 130.268) (width 0.5) (layer B.Cu) (net 1))
   (segment (start 130.955 80.42) (end 133.905 77.47) (width 0.5) (layer B.Cu) (net 1))
   (segment (start 124.592 80.42) (end 130.955 80.42) (width 0.5) (layer B.Cu) (net 1))
   (segment (start 138.43 77.47) (end 133.905 77.47) (width 0.5) (layer B.Cu) (net 1))
   (segment (start 167.875 137.42) (end 168.015 137.42) (width 0.5) (layer B.Cu) (net 1))
-  (segment (start 168.015 137.42) (end 170.815 134.62) (width 0.5) (layer B.Cu) (net 1))
-  (segment (start 170.815 134.62) (end 182.88 134.62) (width 0.5) (layer B.Cu) (net 1))
+  (segment (start 170.53 134.905) (end 170.815 134.62) (width 0.5) (layer B.Cu) (net 1))
+  (segment (start 192.018 130.268) (end 175.167 130.268) (width 0.5) (layer B.Cu) (net 1))
+  (segment (start 168.015 137.42) (end 170.53 134.905) (width 0.5) (layer B.Cu) (net 1))
+  (segment (start 192.018 130.268) (end 210.092 130.268) (width 0.5) (layer B.Cu) (net 1))
+  (segment (start 175.167 130.268) (end 170.53 134.905) (width 0.5) (layer B.Cu) (net 1))
+  (segment (start 189.772 130.268) (end 192.018 130.268) (width 0.5) (layer B.Cu) (net 1))
   (segment (start 67.2 143.65) (end 67.2 144.95) (width 0.5) (layer F.Cu) (net 2))
   (segment (start 69.215 135.255) (end 69.325 135.145) (width 0.5) (layer F.Cu) (net 2))
