File: bottom/left/left-bottom.kicad_pcb (KiCad board)
At the start: 2 copper layers, 137.8 x 95 mm, 7 parts

Commit message: add sign
Parts:
- added G***: LOGO, lib:welcome_to_keyboard_swamp, F.Cu at (137.8, 104.8)
