File: PCB/left/left-PCB.sch (KiCad schematic (older format))
At the start: 43 parts, among them J1 Modulo-Jack, J2 Modulo-Jack, SW1 SW_Push, SW10 SW_Push, SW11 SW_Push, SW12 SW_Push, SW13 SW_Push, SW14 SW_Push, SW15 SW_Push, SW16 SW_Push, SW17 SW_Push, SW18 SW_Push, SW19 SW_Push, SW2 SW_Push, SW20 SW_Push, SW21 SW_Push, SW22 SW_Push, SW23 SW_Push, SW24 SW_Push, SW25 SW_Push, SW26 SW_Push, SW27 SW_Push, SW28 SW_Push, SW3 SW_Push, SW30 SW_Push, SW31 SW_Push, SW32 SW_Push, SW4 SW_Push, SW5 SW_Push, SW50 SW_DIP_x04, SW6 SW_Push, SW7 SW_Push, SW8 SW_Push, SW9 SW_Push, U1 MCP23017_SP, U2 MCP23017_SP

Commit message: change TRRS jack footprint to PJ-320D
Parts:
- J1, J2: footprint lib:TRRS_SMD_SJ2-3574A-SMT_ABCD -> lib:PJ-320D
Changed lines of the file:
@@
 F 0 "J1" H 3132 7067 50  0000 C CNN
 F 1 "Modulo-Jack" H 3132 6976 50  0000 C CNN
-F 2 "lib:TRRS_SMD_SJ2-3574A-SMT_ABCD" H 3425 6875 50  0001 C CNN
+F 2 "lib:PJ-320D" H 3425 6875 50  0001 C CNN
 F 3 "~" H 3425 6875 50  0001 C CNN
 	1    3150 6700
@@
 F 0 "J2" H 4132 7067 50  0000 C CNN
 F 1 "Modulo-Jack" H 4132 6976 50  0000 C CNN
-F 2 "lib:TRRS_SMD_SJ2-3574A-SMT_ABCD" H 4425 6875 50  0001 C CNN
+F 2 "lib:PJ-320D" H 4425 6875 50  0001 C CNN
 F 3 "~" H 4425 6875 50  0001 C CNN
 	1    4150 6700
