File: PCB/right/right-PCB.sch (KiCad schematic (older format))
At the start: 48 parts, among them J1 Modulo-Jack, J2 Modulo-Jack, SW1 SW_Push, SW10 SW_Push, SW11 SW_Push, SW12 SW_Push, SW13 SW_Push, SW14 SW_Push, SW15 SW_Push, SW16 SW_Push, SW17 SW_Push, SW18 SW_Push, SW19 SW_Push, SW2 SW_Push, SW20 SW_Push, SW21 SW_Push, SW22 SW_Push, SW23 SW_Push, SW24 SW_Push, SW25 SW_Push, SW26 SW_Push, SW27 SW_Push, SW28 SW_Push, SW29 SW_Push, SW3 SW_Push, SW30 SW_Push, SW31 SW_Push, SW32 SW_Push, SW33 SW_Push, SW34 SW_Push, SW35 SW_Push, SW36 SW_Push, SW37 SW_Push, SW38 SW_Push, SW4 SW_Push, SW5 SW_Push, SW50 SW_DIP_x04, SW6 SW_Push, SW7 SW_Push, SW8 SW_Push, SW9 SW_Push, U1 MCP23017_SP, U2 MCP23017_SP, U3 MCP23017_SP

Commit message: change TRRS jack footprint to PJ-320D
Parts:
- J1, J2: footprint lib:TRRS_SMD_SJ2-3574A-SMT_ABCD -> lib:PJ-320D
Changed lines of the file:
@@
 F 0 "J1" H 1282 6467 50  0000 C CNN
 F 1 "Modulo-Jack" H 1282 6376 50  0000 C CNN
-F 2 "lib:TRRS_SMD_SJ2-3574A-SMT_ABCD" H 1575 6275 50  0001 C CNN
+F 2 "lib:PJ-320D" H 1575 6275 50  0001 C CNN
 F 3 "~" H 1575 6275 50  0001 C CNN
 	1    1300 6100
@@
 F 0 "J2" H 2382 6467 50  0000 C CNN
 F 1 "Modulo-Jack" H 2382 6376 50  0000 C CNN
-F 2 "lib:TRRS_SMD_SJ2-3574A-SMT_ABCD" H 2675 6275 50  0001 C CNN
+F 2 "lib:PJ-320D" H 2675 6275 50  0001 C CNN
 F 3 "~" H 2675 6275 50  0001 C CNN
 	1    2400 6100
